File: kicad/split_3x_plate.kicad_pcb (KiCad board)
At the start: 2 copper layers, 122.2 x 121.2 mm, 6 parts

Commit message: added svg for acrylic plate cutting
Parts:
- removed G*** (x2): LOGO, graphics:aset
-  : value MountingHole_2.2mm_M2_Pad_Via -> MountingHole_2.2mm_M2; footprint MountingHole:MountingHole_2.2mm_M2_Pad_Via -> MountingHole:MountingHole_2.2mm_M2 (x4)
Other:
- outline, holes or cut-outs redrawn
