File: kicad/split_3x.kicad_pcb (KiCad board)
At the start: 2 copper layers, 127.3 x 121.2 mm, 80 parts, among them SW1 SW_Push, SW2 SW_Push, SW3 Rotary_Encoder_Switch, SW4 Rotary_Encoder_Switch, U1 ProMicro, U2 TRRS

Commit message: modified the silkscreen to work better with the battery
:
Parts:
- added BT1: Bat_loc1, Connector_PinHeader_2.00mm:PinHeader_1x02_P2.00mm_Vertical, F.Cu at (180.7, 74.1)
- added SW5: SW_DIP_x01, other_parts:switch_MSK-12C02_smd, B.Cu at (191.8, 72.8)
- added SW6: SW_DIP_x01, other_parts:switch_MSK-12C02_smd, F.Cu at (191.3, 72.8)
- renumbered spi1 to pim1
Connections:
- U1 pad 24: Net-(U1-Pad24) -> raw
Routing:
- net raw: track 0.00 -> 17.2 mm, vias 0 -> 1
- net Net-(BT1-Pad1): track 0.00 -> 14.4 mm, vias 0 -> 1
- net Net-(U1-Pad24): track 14.4 -> 0.00 mm
- net power: track 515.3 -> 511.4 mm
- net row0: track 135.7 -> 136.5 mm
Other:
- board text added: "GND (blk)"
- board text added: "OFF"
- board text added: "ON"
- board text added: "RAW (red)"

Commit message: added v1.1 silkscreenart, added mangoiv logo, moved the switch footprint a little bit
Parts:
- added G***: LOGO, graphics:mangoiv, B.Cu at (159.3, 55.0)
- added G***: LOGO, graphics:mangoiv, F.Cu at (156.3, 54.0)
- added G***: LOGO, graphics:logo, B.Cu at (190.8, 91.8)
- added G***: LOGO, graphics:logo, F.Cu at (191.9, 91.5)
- moved SW6 1.45 mm to (192.8, 72.8)
Routing:
- net Net-(BT1-Pad1): track 14.4 -> 16.8 mm
- net raw: track 17.2 -> 16.1 mm
Other:
- board text removed: "DracuLad"
- board text removed: "by MangoIV."
